File: Breakout_Board/Breakoutboard_Project.kicad_sch (KiCad schematic)
At the start: 17 parts, among them J1 Conn_01x17, J2 Conn_01x17, J3 Conn_02x06_Top_Bottom, J4 Conn_01x04, U2 STM32F411

Commit message: Swap BMP581 for BMP585, move ADXL interrupts to PB5/PB6, add J4 GND, clean up library pin types
- Add BMP585 library (symbol + LGA9 footprint) and replace U5
- Move ADXL_INT0/INT1 off PA11/PA12 (USB pins) to PB5/PB6
- J4 now 5-pin with GND
- Set GND/VSS pins to power input in ADXL380, MMC5983MA, BMP585 symbols
- Add library prefix to ADXL380 symbol footprint field

Co-Authored-By: Claude Sonnet 5.5 <noreply@anthropic.com>
Parts:
- removed J4: Conn_01x04, Connector_PinSocket_2.54mm:PinSocket_1x04_P2.54mm_Vertical, symbol Connector_Generic:Conn_01x04
- added J4: Conn_01x05, Connector_PinHeader_2.54mm:PinHeader_1x05_P2.54mm_Vertical, symbol Connector_Generic:Conn_01x05
Connections:
- net B5 is gone; now on net ADXL_INT0: J1.13 (Pin_13), U2.13 (B5)
- net B6 is gone; now on net ADXL_INT1: J1.14 (Pin_14), U2.14 (15)
- net ADXL_INT0: no longer J1.8 (Pin_8), U2.8 (A11)
- net ADXL_INT1: no longer J1.9 (Pin_9), U2.9 (A12)
- net Baro_INT: now also J4.2 (Pin_2)
- net CS_BARO: now also J4.4 (Pin_4)
- net CS_MAG: now also J4.3 (Pin_3)
- net GND: now also J4.5 (Pin_5)
- net Mag_INT: now also J4.1 (Pin_1)
- new net A11: J1.8 (Pin_8), U2.8 (A11)
- new net A12: J1.9 (Pin_9), U2.9 (A12)
Changed lines of the file:
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@@
 	(wire
 		(pts
-			(xy 237.49 119.38) (xy 234.95 119.38)
-		)
-		(stroke
-			(width 0)
-			(type default)
-		)
-	)
-	(wire
-		(pts
 			(xy 96.52 30.48) (xy 96.52 27.94)
 		)
@@
 	(wire
 		(pts
-			(xy 237.49 121.92) (xy 234.95 121.92)
-		)
-		(stroke
-			(width 0)
-			(type default)
-		)
-	)
-	(wire
-		(pts
 			(xy 255.27 151.13) (xy 251.46 151.13)
 		)
@@
 	(wire
 		(pts
-			(xy 237.49 116.84) (xy 234.95 116.84)
-		)
-		(stroke
-			(width 0)
-			(type default)
-		)
-	)
-	(wire
-		(pts
 			(xy 184.15 142.24) (xy 181.61 142.24)
 		)
@@
 	(wire
 		(pts
-			(xy 237.49 124.46) (xy 234.95 124.46)
-		)
-		(stroke
-			(width 0)
-			(type default)
-		)
-	)
-	(wire
-		(pts
 			(xy 110.49 74.93) (xy 113.03 74.93)
 		)
@@
 		)
 	)
+	(label "CS_MAG"
+		(at 233.68 121.92 0)
+		(effects
+			(font
+				(size 1.27 1.27)
+			)
+			(justify left bottom)
+		)
+	)
 	(label "A10"
 		(at 82.55 50.8 180)
@@
 		)
 	)
+	(label "CS_BARO"
+		(at 233.68 119.38 0)
+		(effects
+			(font
+				(size 1.27 1.27)
+			)
+			(justify left bottom)
+		)
+	)
 	(label "B7"
 		(at 82.55 71.12 180)
@@
 		)
 	)
-	(label "B5"
+	(label "ADXL_INT0"
 		(at 184.15 129.54 0)
 		(effects
@@
 		)
 	)
-	(label "B6"
+	(label "ADXL_INT1"
 		(at 184.15 127 0)
 		(effects
@@
 		)
 	)
-	(label "CS_MAG"
-		(at 237.49 119.38 0)
-		(effects
-			(font
-				(size 1.27 1.27)
-			)
-			(justify left bottom)
-		)
-	)
 	(label "CS_ADXL"
 		(at 207.01 139.7 0)
@@
 		)
 	)
-	(label "B5"
+	(label "ADXL_INT0"
 		(at 82.55 66.04 180)
 		(effects
@@
 		)
 	)
-	(label "Mag_INT"
-		(at 237.49 124.46 0)
-		(effects
-			(font
-				(size 1.27 1.27)
-			)
-			(justify left bottom)
-		)
-	)
 	(label "A0"
 		(at 113.03 64.77 0)
@@
 		)
 	)
-	(label "CS_BARO"
-		(at 237.49 116.84 0)
-		(effects
-			(font
-				(size 1.27 1.27)
-			)
-			(justify left bottom)
-		)
-	)
 	(label "B9"
 		(at 82.55 76.2 180)
@@
 		)
 	)
-	(label "B6"
+	(label "ADXL_INT1"
 		(at 82.55 68.58 180)
 		(effects
@@
 		)
 	)
-	(label "Baro_INT"
-		(at 237.49 121.92 0)
-		(effects
-			(font
-				(size 1.27 1.27)
-			)
-			(justify left bottom)
-		)
-	)
 	(label "A9"
 		(at 82.55 48.26 180)
@@
 		)
 	)
-	(label "ADXL_INT0"
+	(label "A11"
 		(at 82.55 53.34 180)
 		(effects
@@
 		)
 	)
-	(label "ADXL_INT1"
+	(label "A12"
 		(at 184.15 139.7 0)
 		(effects
@@
 		)
 	)
-	(label "ADXL_INT0"
+	(label "A11"
 		(at 184.15 142.24 0)
 		(effects
@@
 		)
 	)
+	(label "Baro_INT"
+		(at 233.68 124.46 0)
+		(effects
+			(font
+				(size 1.27 1.27)
+			)
+			(justify left bottom)
+		)
+	)
 	(label "CS_ICM"
 		(at 255.27 146.05 0)
@@
 		)
 	)
-	(label "ADXL_INT1"
+	(label "A12"
 		(at 82.55 55.88 180)
 		(effects
@@
 		)
 	)
+	(label "Mag_INT"
+		(at 233.68 127 0)
+		(effects
+			(font
+				(size 1.27 1.27)
+			)
+			(justify left bottom)
+		)
+	)
 	(label "B2"
 		(at 207.01 121.92 0)
@@
 	)
 	(symbol
+		(lib_id "power:GND")
+		(at 233.68 116.84 90)
+		(unit 1)
+		(body_style 1)
+		(exclude_from_sim no)
+		(in_bom yes)
+		(on_board yes)
+		(in_pos_files yes)
+		(dnp no)
+		(fields_autoplaced yes)
+		(property "Reference" "#PWR040"
+			(at 240.03 116.84 0)
+			(hide yes)
+			(show_name no)
+			(do_not_autoplace no)
+			(effects
+				(font
+					(size 1.27 1.27)
+				)
+			)
+		)
+		(property "Value" "GND"
+			(at 237.49 116.8399 90)
+			(show_name no)
+			(do_not_autoplace no)
+			(effects
+				(font
+					(size 1.27 1.27)
+				)
+				(justify right)
+			)
+		)
+		(property "Footprint" ""
+			(at 233.68 116.84 0)
+			(hide yes)
+			(show_name no)
+			(do_not_autoplace no)
+			(effects
+				(font
+					(size 1.27 1.27)
+				)
+			)
+		)
+		(property "Datasheet" ""
+			(at 233.68 116.84 0)
+			(hide yes)
+			(show_name no)
+			(do_not_autoplace no)
+			(effects
+				(font
+					(size 1.27 1.27)
+				)
+			)
+		)
+		(property "Description" "Power symbol creates a global label with name \"GND\" , ground"
+			(at 233.68 116.84 0)
+			(hide yes)
+			(show_name no)
+			(do_not_autoplace no)
+			(effects
+				(font
+					(size 1.27 1.27)
+				)
+			)
+		)
+		(pin "1"
+		)
+		(instances
+			(project "Breakoutboard_Project"
+				(path "/e5b5f554-bb6f-4ecb-9cfb-c4d676c83727"
+					(reference "#PWR040")
+					(unit 1)
+				)
+			)
+		)
+	)
+	(symbol
 		(lib_id "Diode:ESD5Zxx")
 		(at 57.15 83.82 270)
@@
 	)
 	(symbol
+		(lib_id "Connector_Generic:Conn_01x05")
+		(at 228.6 121.92 180)
+		(unit 1)
+		(body_style 1)
+		(exclude_from_sim no)
+		(in_bom yes)
+		(on_board yes)
+		(in_pos_files yes)
+		(dnp no)
+		(fields_autoplaced yes)
+		(property "Reference" "J4"
+			(at 228.6 110.49 0)
+			(show_name no)
+			(do_not_autoplace no)
+			(effects
+				(font
+					(size 1.27 1.27)
+				)
+			)
+		)
+		(property "Value" "Conn_01x05"
+			(at 228.6 113.03 0)
+			(show_name no)
+			(do_not_autoplace no)
+			(effects
+				(font
+					(size 1.27 1.27)
+				)
+			)
+		)
+		(property "Footprint" "Connector_PinHeader_2.54mm:PinHeader_1x05_P2.54mm_Vertical"
+			(at 228.6 121.92 0)
+			(hide yes)
+			(show_name no)
+			(do_not_autoplace no)
+			(effects
+				(font
+					(size 1.27 1.27)
+				)
+			)
+		)
+		(property "Datasheet" ""
+			(at 228.6 121.92 0)
+			(hide yes)
+			(show_name no)
+			(do_not_autoplace no)
+			(effects
+				(font
+					(size 1.27 1.27)
+				)
+			)
+		)
+		(property "Description" "Generic connector, single row, 01x05, script generated (kicad-library-utils/schlib/autogen/connector/)"
+			(at 228.6 121.92 0)
+			(hide yes)
+			(show_name no)
+			(do_not_autoplace no)
+			(effects
+				(font
+					(size 1.27 1.27)
+				)
+			)
+		)
+		(pin "5"
+		)
+		(pin "2"
+		)
+		(pin "4"
+		)
+		(pin "1"
+		)
+		(pin "3"
+		)
+		(instances
+			(project "Breakoutboard_Project"
+				(path "/e5b5f554-bb6f-4ecb-9cfb-c4d676c83727"
+					(reference "J4")
+					(unit 1)
+				)
+			)
+		)
+	)
+	(symbol
 		(lib_id "Connector_Generic:Conn_02x06_Top_Bottom")
 		(at 243.84 148.59 0)
@@
 					(unit 1)
 				)
-			)
-		)
-	)
-	(symbol
-		(lib_id "Connector_Generic:Conn_01x04")
-		(at 229.87 121.92 180)
-		(unit 1)
-		(body_style 1)
-		(exclude_from_sim no)
-		(in_bom yes)
-		(on_board yes)
-		(in_pos_files yes)
-		(dnp no)
-		(fields_autoplaced yes)
-		(property "Reference" "J4"
-			(at 229.87 110.49 0)
-			(show_name no)
-			(do_not_autoplace no)
-			(effects
-				(font
-					(size 1.27 1.27)
-				)
-			)
-		)
-		(property "Value" "Conn_01x04"
-			(at 229.87 113.03 0)
-			(show_name no)
-			(do_not_autoplace no)
-			(effects
-				(font
-					(size 1.27 1.27)
-				)
-			)
-		)
-		(property "Footprint" "Connector_PinSocket_2.54mm:PinSocket_1x04_P2.54mm_Vertical"
-			(at 229.87 121.92 0)
-			(hide yes)
-			(show_name no)
-			(do_not_autoplace no)
-			(effects
-				(font
-					(size 1.27 1.27)
-				)
-			)
-		)
-		(property "Datasheet" ""
-			(at 229.87 121.92 0)
-			(hide yes)
-			(show_name no)
-			(do_not_autoplace no)
-			(effects
-				(font
-					(size 1.27 1.27)
-				)
-			)
-		)
-		(property "Description" "Generic connector, single row, 01x04, script generated (kicad-library-utils/schlib/autogen/connector/)"
-			(at 229.87 121.92 0)
-			(hide yes)
-			(show_name no)
-			(do_not_autoplace no)
-			(effects
-				(font
-					(size 1.27 1.27)
-				)
-			)
-		)
-		(pin "4"
-		)
-		(pin "2"
-		)
-		(pin "3"
-		)
-		(pin "1"
-		)
-		(instances
-			(project "Breakoutboard_Project"
-				(path "/e5b5f554-bb6f-4ecb-9cfb-c4d676c83727"
-					(reference "J4")
-					(unit 1)
-				)
