File: Breakout_Board/Breakoutboard_Project.kicad_sch (KiCad schematic)
At the start: 17 parts, among them J1 Conn_01x17, J2 Conn_01x17, J3 Conn_02x06_Top_Bottom, J4 Conn_01x05, U2 STM32F411

Commit message: small chagneds
Connections:
- net B0 is gone; now on net CS_MAG: J2.14 (Pin_14), U2.34 (B0)
- net CS_MAG: no longer J2.7 (Pin_7), U2.27 (A1)
- new net A1: J2.7 (Pin_7), U2.27 (A1)
Changed lines of the file:
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@@
+		)
+	)
+	(label "CS_MAG"
+		(at 207.01 127 0)
+		(effects
+			(font
+				(size 1.27 1.27)
+			)
+			(justify left bottom)
 		)
 	)
@@
 		)
 	)
-	(label "CS_MAG"
-		(at 114.3 62.23 0)
-		(effects
-			(font
-				(size 1.27 1.27)
-			)
-			(justify left bottom)
-		)
-	)
 	(label "CS_BARO"
 		(at 233.68 119.38 0)
@@
 		)
 	)
+	(label "A1"
+		(at 207.01 144.78 0)
+		(effects
+			(font
+				(size 1.27 1.27)
+			)
+			(justify left bottom)
+		)
+	)
 	(label "ICM_INT1"
 		(at 233.68 156.21 180)
@@
 		)
 	)
-	(label "B0"
-		(at 113.03 44.45 0)
-		(effects
-			(font
-				(size 1.27 1.27)
-			)
-			(justify left bottom)
-		)
-	)
 	(label "CS_ADXL"
 		(at 255.27 143.51 0)
@@
 		)
 	)
+	(label "CS_MAG"
+		(at 113.03 44.45 0)
+		(effects
+			(font
+				(size 1.27 1.27)
+			)
+			(justify left bottom)
+		)
+	)
 	(label "B12"
 		(at 184.15 160.02 0)
@@
 		)
 	)
-	(label "CS_MAG"
-		(at 207.01 144.78 0)
-		(effects
-			(font
-				(size 1.27 1.27)
-			)
-			(justify left bottom)
-		)
-	)
 	(label "MOSI"
 		(at 34.29 134.62 180)
@@
 		)
 	)
-	(label "B0"
-		(at 207.01 127 0)
-		(effects
-			(font
-				(size 1.27 1.27)
-			)
-			(justify left bottom)
-		)
-	)
 	(label "A9"
 		(at 82.55 48.26 180)
@@
 		(effects
 			(font
+				(size 1.27 1.27)
+			)
+			(justify left bottom)
+		)
+	)
+	(label "A1"
+		(at 114.3 62.23 0)
+		(effects
+			(font

Commit message: minor
Connections:
- net Baro_INT: now also J4.3 (Pin_3); no longer J4.2 (Pin_2)
- net CS_MAG: now also J4.2 (Pin_2); no longer J4.3 (Pin_3)
Changed lines of the file:
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@@
-		)
-	)
-	(label "CS_MAG"
-		(at 233.68 121.92 0)
-		(effects
-			(font
-				(size 1.27 1.27)
-			)
-			(justify left bottom)
 		)
 	)
@@
 		)
 	)
+	(label "Baro_INT"
+		(at 233.68 121.92 0)
+		(effects
+			(font
+				(size 1.27 1.27)
+			)
+			(justify left bottom)
+		)
+	)
 	(label "ADXL_INT1"
 		(at 196.85 39.37 180)
@@
 		)
 	)
+	(label "CS_MAG"
+		(at 233.68 124.46 0)
+		(effects
+			(font
+				(size 1.27 1.27)
+			)
+			(justify left bottom)
+		)
+	)
 	(label "A8"
 		(at 82.55 45.72 180)
@@
 		(effects
 			(font
-				(size 1.27 1.27)
-			)
-			(justify left bottom)
-		)
-	)
-	(label "Baro_INT"
-		(at 233.68 124.46 0)
-		(effects
-			(font

Commit message: PCB finished
Parts:
- removed J3: Conn_02x06_Top_Bottom, Connector_Hirose:Hirose_DF11-12DP-2DSA_2x06_P2.00mm_Vertical, symbol Connector_Generic:Conn_02x06_Top_Bottom
- removed J4: Conn_01x05, Connector_PinHeader_2.54mm:PinHeader_1x05_P2.54mm_Vertical, symbol Connector_Generic:Conn_01x05
Connections:
- net B10 is gone; now on net Mag_INT: J2.17 (Pin_17), U2.37 (B10)
- net B7 is gone; now on net ICM_INT1: J1.15 (Pin_15), U2.15 (B7)
- net C14 is gone; now on net CS_ADXL: J2.3 (Pin_3), U2.23 (C14)
- net ADXL_INT0: now also J1.14 (Pin_14), U2.14 (15); no longer J1.13 (Pin_13), U2.13 (B5)
- net ADXL_INT1: now also J1.13 (Pin_13), U2.13 (B5); no longer J1.14 (Pin_14), U2.14 (15)
- net CS_ADXL: no longer J2.9 (Pin_9), U2.29 (A3)
- net CS_BARO: now also J2.10 (Pin_10), U2.30 (A4); no longer J2.8 (Pin_8), U2.28 (A2)
- net CS_ICM: now also J2.8 (Pin_8), U2.28 (A2); no longer J2.10 (Pin_10), U2.30 (A4)
- net ICM_INT1: no longer J1.10 (Pin_10), U2.10 (A15)
- net Mag_INT: no longer J1.3 (Pin_3), U2.3 (B14)
- new net A15: J1.10 (Pin_10), U2.10 (A15)
- new net A3: J2.9 (Pin_9), U2.29 (A3)
- new net B14: J1.3 (Pin_3), U2.3 (B14)
Other:
- note removed: "J3 Accel/Gyro"
- note removed: "J4 Mag/Bar"
