File: Breakout_Board/Accel_Gyro.kicad_sch (KiCad schematic)
At the start: 10 parts, among them U1 ADXL380-2BCCZ-RL7, U3 ICM-40609-D

Commit message: Swap BMP581 for BMP585, move ADXL interrupts to PB5/PB6, add J4 GND, clean up library pin types
- Add BMP585 library (symbol + LGA9 footprint) and replace U5
- Move ADXL_INT0/INT1 off PA11/PA12 (USB pins) to PB5/PB6
- J4 now 5-pin with GND
- Set GND/VSS pins to power input in ADXL380, MMC5983MA, BMP585 symbols
- Add library prefix to ADXL380 symbol footprint field

Co-Authored-By: Claude Sonnet 5.5 <noreply@anthropic.com>
Connections:
- no-connect marks 2 -> 3
Changed lines of the file:
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@@
+	)
+	(no_connect
+		(at 96.52 30.48)
 	)
 	(no_connect
