File: Breakout_Board/Accel_Gyro.kicad_sch (KiCad schematic)
At the start: 10 parts, among them U1 ADXL380-2BCCZ-RL7, U3 ICM-40609-D

Commit message: updadetd shcematic stuff
Other:
- note removed: "These are external clocks"
- note removed: "ensure what bclk mclk and other stuff do here?"
Changed lines of the file:
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@@
 	(generator_version "10.0")
 	(paper "A4")
-	(text "ensure what bclk mclk and other stuff do here?\n"
-		(exclude_from_sim no)
-		(at 76.454 53.34 0)
-		(effects
-			(font
-				(size 1.27 1.27)
-				(thickness 0.254)
-				(bold yes)
-			)
-		)
-	)
-	(text "These are external clocks"
-		(exclude_from_sim no)
-		(at 99.314 23.114 0)
-		(effects
-			(font
-				(size 1.016 1.016)
-			)
-		)
-	)
 	(junction
 		(at 220.98 16.51)
