File: Breakout_Board/Breakoutboard_Project.kicad_pcb (KiCad board)
At the start: 2 copper layers, 60 x 60 mm, 36 parts, among them J1 Conn_01x17, J2 Conn_01x17, J3 Conn_02x06_Top_Bottom, J4 Conn_01x04, U1 ADXL380-2BCCZ-RL7, U2 STM32F411, U3 ICM-40609-D, U4 MMC5983MA, U5 BMP581

Commit message: Swap BMP581 for BMP585, move ADXL interrupts to PB5/PB6, add J4 GND, clean up library pin types
- Add BMP585 library (symbol + LGA9 footprint) and replace U5
- Move ADXL_INT0/INT1 off PA11/PA12 (USB pins) to PB5/PB6
- J4 now 5-pin with GND
- Set GND/VSS pins to power input in ADXL380, MMC5983MA, BMP585 symbols
- Add library prefix to ADXL380 symbol footprint field

Co-Authored-By: Claude Sonnet 5.5 <noreply@anthropic.com>
Connections:
- J1 pad 13: /B5 -> /ADXL_INT0
- J1 pad 14: /B6 -> /ADXL_INT1
- J1 pad 8: /ADXL_INT0 -> /A11
- J1 pad 9: /ADXL_INT1 -> /A12
- U2 pad 13: /B5 -> /ADXL_INT0
- U2 pad 14: /B6 -> /ADXL_INT1
- U2 pad 8: /ADXL_INT0 -> /A11
- U2 pad 9: /ADXL_INT1 -> /A12
Routing:
- net /B6: track 5.12 -> 0.00 mm
- net /B5: track 5.12 -> 0.00 mm
- net /A12: track 0.00 -> 4.32 mm
- net /A11: track 0.00 -> 4.32 mm
- net /ADXL_INT1: track 4.32 -> 5.12 mm
- net /ADXL_INT0: track 4.32 -> 5.12 mm

Commit message: Save PCB with BMP585 (U5) and 5-pin J4 footprints
Co-Authored-By: Claude Sonnet 5.5 <noreply@anthropic.com>
Parts:
- added J4: Conn_01x05, Connector_PinHeader_2.54mm:PinHeader_1x05_P2.54mm_Vertical, F.Cu at (86.8, 42.8)
- U5: value BMP581 -> BMP585; footprint BMP581:QFN10_BMP581_BOS -> BMP585:LGA9_BMP585_BOS
Connections:
- U5 pad 1: +3.3V -> /SCLK
- U5 pad 2: /SCLK -> /MOSI
- U5 pad 3: GND -> /MISO
- U5 pad 4: /MOSI -> +3.3V
- U5 pad 5: /MISO -> /Baro_INT
- U5 pad 6: /CS_BARO -> GND
- U5 pad 7: /Baro_INT -> /CS_BARO
- U5 pad 8: GND -> +3.3V
- U5 pad 9: GND -> unconnected-(U5-L/M-Pad9)
