File: Breakout_Board/Breakoutboard_Project.kicad_pcb (KiCad board)
At the start: 2 copper layers, 60 x 60 mm, 37 parts, among them J1 Conn_01x17, J2 Conn_01x17, J3 Conn_02x06_Top_Bottom, J4 Conn_01x04, J4 Conn_01x05, U1 ADXL380-2BCCZ-RL7, U2 STM32F411, U3 ICM-40609-D, U4 MMC5983MA, U5 BMP585

Commit message: small chagneds
Parts:
- moved J4 16.6 mm to (70.3, 44.7)
Connections:
- J2 pad 14: /B0 -> /CS_MAG
- J2 pad 7: /CS_MAG -> /A1
- U2 pad 27: /CS_MAG -> /A1
- U2 pad 34: /B0 -> /CS_MAG
Routing:
- net /B0: track 4.82 -> 0.00 mm
- net /A1: track 0.00 -> 4.82 mm

Commit message: minor
Parts:
- removed the J4 at (74.6, 44.7)
- moved J4 4.26 mm to (74.6, 44.5)
Connections:
- J4 pad 2: /Baro_INT -> /CS_MAG
- J4 pad 3: /CS_MAG -> /Baro_INT
Routing:
- net +5V: track 36.3 -> 104.8 mm
- net /MISO: track 4.82 -> 58.0 mm, vias 0 -> 1
- net /Baro_INT: track 4.32 -> 55.4 mm
- net /SCLK: track 4.82 -> 49.2 mm, vias 0 -> 2
- net /MOSI: track 4.82 -> 43.1 mm, vias 0 -> 1
- net /CS_MAG: track 4.82 -> 38.2 mm
- net /CS_BARO: track 4.82 -> 33.0 mm
- net +3.3V: track 16.8 -> 34.0 mm, vias 0 -> 4
- net /Mag_INT: track 4.32 -> 18.3 mm
- net GND: track 44.0 -> 56.4 mm, vias 2 -> 8

Commit message: Update Breakoutboard_Project.kicad_pcb
Routing:
- net /SCLK: track 49.2 -> 45.3 mm
Changed lines of the file:
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@@
 	)
 	(segment
+		(start 75.75 45.85)
+		(end 74.6 47)
+		(width 0.2)
+		(layer "F.Cu")
+		(net "/CS_MAG")
+	)
+	(segment
+		(start 48.091244 49.49)
+		(end 48.058744 49.4575)
+		(width 0.2)
+		(layer "F.Cu")
+		(net "/CS_MAG")
+	)
+	(segment
+		(start 52.868744 49.49)
+		(end 72.11 49.49)
+		(width 0.2)
+		(layer "F.Cu")
+		(net "/CS_MAG")
+	)
+	(segment
+		(start 75.075002 37.154999)
+		(end 75.75 37.829997)
+		(width 0.2)
+		(layer "F.Cu")
+		(net "/CS_MAG")
+	)
+	(segment
+		(start 75.75 37.829997)
+		(end 75.75 45.85)
+		(width 0.2)
+		(layer "F.Cu")
+		(net "/CS_MAG")
+	)
+	(segment
+		(start 52.868744 49.49)
+		(end 48.091244 49.49)
+		(width 0.2)
+		(layer "F.Cu")
+		(net "/CS_MAG")
+	)
+	(segment
+		(start 72.11 49.49)
+		(end 74.6 47)
+		(width 0.2)
+		(layer "F.Cu")
+		(net "/CS_MAG")
+	)
+	(segment
 		(start 28.678744 36.7575)
 		(end 24.381244 36.7575)
@@
 	)
 	(segment
-		(start 75.75 45.85)
-		(end 74.6 47)
-		(width 0.2)
-		(layer "F.Cu")
-		(net "/CS_MAG")
-	)
-	(segment
-		(start 48.091244 49.49)
-		(end 48.058744 49.4575)
-		(width 0.2)
-		(layer "F.Cu")
-		(net "/CS_MAG")
-	)
-	(segment
-		(start 52.868744 49.49)
-		(end 72.11 49.49)
-		(width 0.2)
-		(layer "F.Cu")
-		(net "/CS_MAG")
-	)
-	(segment
-		(start 75.075002 37.154999)
-		(end 75.75 37.829997)
-		(width 0.2)
-		(layer "F.Cu")
-		(net "/CS_MAG")
-	)
-	(segment
-		(start 75.75 37.829997)
-		(end 75.75 45.85)
-		(width 0.2)
-		(layer "F.Cu")
-		(net "/CS_MAG")
-	)
-	(segment
-		(start 52.868744 49.49)
-		(end 48.091244 49.49)
-		(width 0.2)
-		(layer "F.Cu")
-		(net "/CS_MAG")
-	)
-	(segment
-		(start 72.11 49.49)
-		(end 74.6 47)
-		(width 0.2)
-		(layer "F.Cu")
-		(net "/CS_MAG")
-	)
-	(segment
 		(start 63.508799 60.1)
 		(end 62.426999 59.0182)
@@
 	)
 	(segment
-		(start 65.2 40.8)
-		(end 54.25 51.75)
-		(width 0.2)
-		(layer "B.Cu")
-		(net "/SCLK")
-	)
-	(segment
 		(start 62.5 55.251471)
 		(end 61.598529 54.35)
@@
 	)
 	(segment
-		(start 54.25 55.728744)
-		(end 52.868744 57.11)
+		(start 73.1 38.55)
+		(end 72.6 38.55)
 		(width 0.2)
 		(layer "B.Cu")
@@
 	)
 	(segment
-		(start 70.35 40.8)
-		(end 65.2 40.8)
+		(start 72.6 38.55)
+		(end 70.35 40.8)
 		(width 0.2)
 		(layer "B.Cu")
@@
 	)
 	(segment
-		(start 73.1 38.55)
-		(end 72.6 38.55)
+		(start 65.2 40.8)
+		(end 55.628744 50.371256)
 		(width 0.2)
 		(layer "B.Cu")
@@
 	)
 	(segment
-		(start 72.6 38.55)
-		(end 70.35 40.8)
+		(start 70.35 40.8)
+		(end 65.2 40.8)
 		(width 0.2)
 		(layer "B.Cu")
@@
 	)
 	(segment
-		(start 54.25 51.75)
-		(end 54.25 55.728744)
+		(start 55.628744 50.371256)
+		(end 55.628744 54.35)
 		(width 0.2)
 		(layer "B.Cu")
@@
 	)
 	(segment
-		(start 51.718744 57.586346)
-		(end 51.718744 55.72)
+		(start 56.7 54.95)
+		(end 53.39 58.26)
 		(width 0.2)
 		(layer "B.Cu")
@@
 	)
 	(segment
-		(start 51.718744 55.72)
-		(end 52.868744 54.57)
+		(start 52.392398 58.26)
+		(end 51.718744 57.586346)
 		(width 0.2)
 		(layer "B.Cu")
@@
 	)
 	(segment
-		(start 61.35 54.95)
-		(end 58.04 58.26)
+		(start 53.39 58.26)
+		(end 52.392398 58.26)
 		(width 0.2)
 		(layer "B.Cu")
@@
 	)
 	(segment
-		(start 52.392398 58.26)
-		(end 51.718744 57.586346)
+		(start 51.718744 57.586346)
+		(end 51.718744 55.72)
 		(width 0.2)
 		(layer "B.Cu")
@@
 	)
 	(segment
-		(start 58.04 58.26)
-		(end 52.392398 58.26)
+		(start 61.35 54.95)
+		(end 56.7 54.95)
+		(width 0.2)
+		(layer "B.Cu")
+		(net "/MISO")
+	)
+	(segment
+		(start 51.718744 55.72)
+		(end 52.868744 54.57)
 		(width 0.2)
 		(layer "B.Cu")
@@
 		(layer "F.Cu")
 		(hatch none 0.1)
-		(priority 30081)
+		(priority 30080)
 		(attr
 			(teardrop
@@
 		(polygon
 			(pts
-				(xy 61.7125 33.1175) (xy 61.620011 33.098931) (xy 61.522135 33.040583) (xy 61.410739 32.945702)
-				(xy 61.226335 32.792773) (xy 61.109685 32.717228) (xy 60.970671 32.64903) (xy 60.399 33.2175) (xy 60.970671 33.78597)
-				(xy 61.153545 33.691455) (xy 61.320629 33.568214) (xy 61.410739 33.489298) (xy 61.56079 33.367256)
-				(xy 61.634138 33.33079) (xy 61.7125 33.3175)
+				(xy 59.0875 33.3175) (xy 59.179989 33.336069) (xy 59.277865 33.394417) (xy 59.389261 33.489298)
+				(xy 59.573665 33.642227) (xy 59.690315 33.717772) (xy 59.829329 33.78597) (xy 60.401 33.2175) (xy 59.829329 32.64903)
+				(xy 59.646455 32.743545) (xy 59.479371 32.866786) (xy 59.389261 32.945702) (xy 59.23921 33.067744)
+				(xy 59.165862 33.10421) (xy 59.0875 33.1175)
 			)
 		)
@@
 		(layer "F.Cu")
 		(hatch none 0.1)
-		(priority 30080)
+		(priority 30081)
 		(attr
 			(teardrop
@@
 		(polygon
 			(pts
-				(xy 59.0875 33.3175) (xy 59.179989 33.336069) (xy 59.277865 33.394417) (xy 59.389261 33.489298)
-				(xy 59.573665 33.642227) (xy 59.690315 33.717772) (xy 59.829329 33.78597) (xy 60.401 33.2175) (xy 59.829329 32.64903)
-				(xy 59.646455 32.743545) (xy 59.479371 32.866786) (xy 59.389261 32.945702) (xy 59.23921 33.067744)
-				(xy 59.165862 33.10421) (xy 59.0875 33.1175)
+				(xy 61.7125 33.1175) (xy 61.620011 33.098931) (xy 61.522135 33.040583) (xy 61.410739 32.945702)
+				(xy 61.226335 32.792773) (xy 61.109685 32.717228) (xy 60.970671 32.64903) (xy 60.399 33.2175) (xy 60.970671 33.78597)
+				(xy 61.153545 33.691455) (xy 61.320629 33.568214) (xy 61.410739 33.489298) (xy 61.56079 33.367256)
+				(xy 61.634138 33.33079) (xy 61.7125 33.3175)
 			)
 		)
@@
 	)
 	(zone
-		(net "/MISO")
+		(net "/MOSI")
 		(layer "B.Cu")
 		(hatch none 0.1)
-		(priority 30003)
+		(priority 30001)
 		(attr
 			(teardrop
@@
 		(polygon
 			(pts
-				(xy 51.818744 55.789562) (xy 51.818744 55.72) (xy 51.789455 55.790711) (xy 51.890562 55.696508)
-				(xy 51.9836 55.623512) (xy 52.064987 55.571907) (xy 52.142366 55.534121) (xy 52.293624 55.490337)
-				(xy 52.477416 55.473481) (xy 52.527118 55.471663) (xy 52.78467 55.454221) (xy 52.938831 55.428732)
-				(xy 53.115486 55.383399) (xy 52.872345 54.566399) (xy 52.055345 54.323258) (xy 51.994859 54.581589)
-				(xy 51.970572 54.823442) (xy 51.967081 54.911627) (xy 51.956267 55.090512) (xy 51.942414 55.175686)
-				(xy 51.918242 55.261029) (xy 51.880235 55.348799) (xy 51.824875 55.441259) (xy 51.748647 55.540669)
-				(xy 51.648033 55.649289) (xy 51.618744 55.72) (xy 51.618744 55.789562)
+				(xy 53.997221 50.760102) (xy 53.8894 50.861006) (xy 53.790634 50.939641) (xy 53.705021 50.995454)
+				(xy 53.623792 51.036984) (xy 53.465885 51.087261) (xy 53.274402 51.111391) (xy 53.218237 51.11541)
+				(xy 52.957169 51.141044) (xy 52.800877 51.169643) (xy 52.622002 51.216601) (xy 52.865143 52.033601)
+				(xy 53.682143 52.276742) (xy 53.748316 52.000328) (xy 53.779078 51.740018) (xy 53.783334 51.680507)
+				(xy 53.801228 51.491023) (xy 53.818642 51.401363) (xy 53.846643 51.311679) (xy 53.888937 51.219412)
+				(xy 53.949231 51.122003) (xy 54.03123 51.016893) (xy 54.138642 50.901523)
 			)
 		)
 	)
 	(zone
-		(net "/SCLK")
+		(net "GND")
 		(layer "B.Cu")
-		(hatch none 0.1)
-		(priority 30001)
-		(attr
-			(teardrop
-				(type padvia)
-			)
-		)
-		(connect_pads yes
-			(clearance 0)
+		(name "gnd")
+		(hatch edge 0.5)
+		(priority 1)
+		(connect_pads
+			(clearance 0.5)
 		)
-		(min_thickness 0.0254)
+		(min_thickness 0.25)
 		(fill yes
-			(island_removal_mode 1)
+			(thermal_gap 0.5)
+			(thermal_bridge_width 0.5)
+			(island_removal_mode 0)
 		)
 		(polygon
 			(pts
-				(xy 53.997221 55.840102) (xy 53.8894 55.941006) (xy 53.790634 56.019641) (xy 53.705021 56.075454)
-				(xy 53.623792 56.116984) (xy 53.465885 56.167261) (xy 53.274402 56.191391) (xy 53.218237 56.19541)
-				(xy 52.957169 56.221044) (xy 52.800877 56.249643) (xy 52.622002 56.296601) (xy 52.865143 57.113601)
-				(xy 53.682143 57.356742) (xy 53.748316 57.080328) (xy 53.779078 56.820018) (xy 53.783334 56.760507)
-				(xy 53.801228 56.571023) (xy 53.818642 56.481363) (xy 53.846643 56.391679) (xy 53.888937 56.299412)
-				(xy 53.949231 56.202003) (xy 54.03123 56.096893) (xy 54.138642 55.981523)
+				(xy 14.952108 26.982164) (xy 89.732108 26.982164) (xy 89.169354 97.326394) (xy 13.827092 96.733148)
 			)
 		)
 	)
 	(zone
-		(net "/MOSI")
+		(net "/MISO")
 		(layer "B.Cu")
 		(hatch none 0.1)
@@
 		(polygon
 			(pts
-				(xy 53.997221 50.760102) (xy 53.8894 50.861006) (xy 53.790634 50.939641) (xy 53.705021 50.995454)
-				(xy 53.623792 51.036984) (xy 53.465885 51.087261) (xy 53.274402 51.111391) (xy 53.218237 51.11541)
-				(xy 52.957169 51.141044) (xy 52.800877 51.169643) (xy 52.622002 51.216601) (xy 52.865143 52.033601)
-				(xy 53.682143 52.276742) (xy 53.748316 52.000328) (xy 53.779078 51.740018) (xy 53.783334 51.680507)
-				(xy 53.801228 51.491023) (xy 53.818642 51.401363) (xy 53.846643 51.311679) (xy 53.888937 51.219412)
-				(xy 53.949231 51.122003) (xy 54.03123 51.016893) (xy 54.138642 50.901523)
-			)
-		)
-	)
-	(zone
-		(net "GND")
-		(layer "B.Cu")
-		(name "gnd")
-		(hatch edge 0.5)
-		(priority 1)
-		(connect_pads
-			(clearance 0.5)
-		)
-		(min_thickness 0.25)
-		(fill yes
-			(thermal_gap 0.5)
-			(thermal_bridge_width 0.5)
-			(island_removal_mode 0)
-		)
-		(polygon
-			(pts
-				(xy 14.952108 26.982164) (xy 89.732108 26.982164) (xy 89.169354 97.326394) (xy 13.827092 96.733148)
+				(xy 51.818744 55.789562) (xy 51.818744 55.72) (xy 51.789455 55.790711) (xy 51.890562 55.696508)
+				(xy 51.9836 55.623512) (xy 52.064987 55.571907) (xy 52.142366 55.534121) (xy 52.293624 55.490337)
+				(xy 52.477416 55.473481) (xy 52.527118 55.471663) (xy 52.78467 55.454221) (xy 52.938831 55.428732)
+				(xy 53.115486 55.383399) (xy 52.872345 54.566399) (xy 52.055345 54.323258) (xy 51.994859 54.581589)
+				(xy 51.970572 54.823442) (xy 51.967081 54.911627) (xy 51.956267 55.090512) (xy 51.942414 55.175686)
+				(xy 51.918242 55.261029) (xy 51.880235 55.348799) (xy 51.824875 55.441259) (xy 51.748647 55.540669)
+				(xy 51.648033 55.649289) (xy 51.618744 55.72) (xy 51.618744 55.789562)
 			)
 		)

Commit message: PCB finished
Parts:
- removed J3: Conn_02x06_Top_Bottom, Connector_Hirose:Hirose_DF11-12DP-2DSA_2x06_P2.00mm_Vertical
- removed J4: Conn_01x05, Connector_PinHeader_2.54mm:PinHeader_1x05_P2.54mm_Vertical
- moved R2 12.7 mm to (60.5, 37.2)
- moved D6 12.7 mm to (60.5, 33.1)
- moved R1 12.5 mm to (62.8, 37.2)
- moved D7 12.5 mm to (62.8, 33.2)
- moved G*** 11.9 mm to (74.2, 74.0)
- moved C10 8.80 mm to (75.0, 39.5), turned to 0 degrees
- moved C20 8.80 mm to (75.0, 33.3), turned to 0 degrees
- moved D5 7.27 mm to (70.9, 33.1), turned to 180 degrees
- moved C22 6.25 mm to (75.0, 36.3), turned to 0 degrees
- moved C3 6.09 mm to (57.4, 38.0)
- moved C6 6.06 mm to (57.4, 33.4)
- moved C5 5.31 mm to (55.2, 33.4)
- moved C2 5.18 mm to (55.3, 38.0)
- moved C18 4.69 mm to (67.9, 53.9)
- moved C16 4.69 mm to (67.9, 50.7)
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Connections:
- J1 pad 10: /ICM_INT1 -> /A15
- J1 pad 13: /ADXL_INT0 -> /ADXL_INT1
- J1 pad 14: /ADXL_INT1 -> /ADXL_INT0
- J1 pad 15: /B7 -> /ICM_INT1
- J1 pad 3: /Mag_INT -> /B14
- J2 pad 10: /CS_ICM -> /CS_BARO
- J2 pad 17: /B10 -> /Mag_INT
- J2 pad 3: /C14 -> /CS_ADXL
- J2 pad 8: /CS_BARO -> /CS_ICM
- J2 pad 9: /CS_ADXL -> /A3
- U2 pad 10: /ICM_INT1 -> /A15
- U2 pad 13: /ADXL_INT0 -> /ADXL_INT1
- U2 pad 14: /ADXL_INT1 -> /ADXL_INT0
- U2 pad 15: /B7 -> /ICM_INT1
- U2 pad 23: /C14 -> /CS_ADXL
- U2 pad 28: /CS_BARO -> /CS_ICM
- U2 pad 29: /CS_ADXL -> /A3
- U2 pad 3: /Mag_INT -> /B14
- U2 pad 30: /CS_ICM -> /CS_BARO
- U2 pad 37: /B10 -> /Mag_INT
Routing:
- net /FSYNC_ADXL: track 5.12 -> 94.1 mm
- net /MOSI: track 43.1 -> 107.0 mm, vias 1 -> 0
- net /ADXL_INT1: track 5.12 -> 65.7 mm
- net /ADXL_INT0: track 5.12 -> 61.1 mm
- net /MISO: track 58.0 -> 103.7 mm, vias 1 -> 5
- net /ICM_INT1: track 4.32 -> 42.2 mm, vias 0 -> 2
- net +5V: track 104.8 -> 67.0 mm, vias 0 -> 2
- net /FSYNC_ICM: track 4.32 -> 39.6 mm, vias 0 -> 2
- net +3.3V: track 34.0 -> 65.6 mm, vias 4 -> 13
- net /Baro_INT: track 55.4 -> 86.8 mm, vias 0 -> 2
- net /SCLK: track 45.3 -> 75.2 mm, vias 2 -> 5
- net GND: track 56.4 -> 42.9 mm, vias 8 -> 24
- net /Mag_INT: track 18.3 -> 30.6 mm
- net /CS_ADXL: track 4.82 -> 15.0 mm
- net /CS_MAG: track 38.2 -> 28.5 mm
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